File: kicad/choc/horizon-choc.kicad_pcb (KiCad board)
At the start: 2 copper layers, 252 x 68 mm, 116 parts, among them SW1 SW_Push, SW10 SW_Push, SW11 SW_Push, SW12 SW_Push, SW13 SW_Push, SW14 SW_Push, SW15 SW_Push, SW16 SW_Push, SW17 SW_Push, SW18 SW_Push, SW19 SW_Push, SW2 SW_Push, SW20 SW_Push, SW21 SW_Push, SW22 SW_Push, SW23 SW_Push, SW24 SW_Push, SW25 SW_Push, SW26 SW_Push, SW27 SW_Push, SW28 SW_Push, SW29 SW_Push, SW3 SW_Push, SW30 SW_Push, SW31 SW_Push, SW32 SW_Push, SW33 SW_Push, SW34 SW_Push, SW35 SW_Push, SW36 SW_Push, SW37 SW_Push, SW38 SW_Push, SW39 SW_Push, SW4 SW_Push, SW40 SW_Push, SW41 SW_Push, SW42 SW_Push, SW43 SW_Push, SW44 SW_Push, SW45 SW_Push, SW46 SW_Push, SW47 SW_Push, SW48 SW_Push, SW49 SW_Push, SW5 SW_Push, SW50 SW_Push, SW51 SW_Push, SW52 SW_Push, SW6 SW_Push, SW7 SW_Push, SW8 SW_Push, SW9 SW_Push, U1 PRO-MICRO

Commit message: Add files via upload
Parts:
- added H1: Hole_Pad, horizon-footprints:Mount_M2, F.Cu at (2.50, 2.50)
- added H2: Hole_Pad, horizon-footprints:Mount_M2, F.Cu at (2.50, 8.50)
- added H3: Hole_Pad, horizon-footprints:Mount_M2, F.Cu at (8.50, 2.50)
- added H4: Hole_Pad, horizon-footprints:Mount_M2, F.Cu at (8.50, 8.50)
- added H5: Hole_Pad, horizon-footprints:Mount_M2, F.Cu at (14.5, 2.50)
- added H6: Hole_Pad, horizon-footprints:Mount_M2, F.Cu at (14.5, 8.50)
- added H7: Hole_Pad, horizon-footprints:Mount_M2, F.Cu at (20.5, 2.50)
- added H8: Hole_Pad, horizon-footprints:Mount_M2, F.Cu at (20.5, 8.50)
Routing:
- net COL14: track 183.5 -> 210.7 mm
- net COL12: track 143.3 -> 170.4 mm
- net COL13: track 163.4 -> 190.6 mm
- net COL11: track 123.2 -> 150.3 mm
- net COL10: track 104.1 -> 131.3 mm
- net COL9: track 85.1 -> 112.2 mm
- net COL1: track 183.5 -> 204.5 mm
- net COL6: track 85.1 -> 104.2 mm
- net COL4: track 123.2 -> 142.3 mm
- net COL2: track 163.4 -> 182.6 mm
- net COL3: track 143.3 -> 162.4 mm
- net COL5: track 104.1 -> 121.4 mm
- net COL8: track 24.9 -> 25.9 mm
- net COL7: track 24.9 -> 25.9 mm

Commit message: Add files via upload
Parts:
- removed H1, H2, H3, H4, H5, H6, H7, H8: Hole_Pad, horizon-footprints:Mount_M2
Routing:
- net COL5: track 121.4 -> 123.3 mm
